Commit message: urdf

File: examples/2_link.urdf.xacro (robot description, xacro)
@@ -1,5 +1,6 @@
 <?xml version="1.0" ?>
-<robot name="2_link" xmlns:xacro="http://www.ros.org/wiki/xacro">    <xacro:macro name="inertial_cylinder" params="mass length radius *origin">
-        <inertial>
+<robot name="2_link" xmlns:xacro="http://www.ros.org/wiki/xacro">
+    <xacro:macro name="inertial_cylinder" params="mass length radius *origin">
+    <inertial>
             <xacro:insert_block name="origin"/>
             <mass value="${mass}" />
@@ -8,9 +9,13 @@
                     izz="${(1/2) * mass * (radius*radius)}" />
         </inertial>
-    </xacro:macro>    <link name="base_link"></link>    <joint name="joint1" type="continuous">        <parent link="base_link"/>
+    </xacro:macro>
+    <link name="base_link"></link>
+    <joint name="joint1" type="continuous">
+         <parent link="base_link"/>
         <child link="link1"/>
         <origin xyz="0 0 0 " rpy="0 0 0"/>
         <axis xyz="0 1 0" />
-    </joint>    <link name="link1">
+    </joint>
+    <link name="link1">
         <xacro:inertial_cylinder mass="0.1" length="1.0" radius="0.05">
             <origin xyz="0 0 0.5" rpy="0 0 0"/>
@@ -28,9 +33,11 @@
             </geometry>
         </collision>
-    </link>    <joint name="joint2" type="continuous">        <parent link="link1"/>
+    </link>
+    <joint name="joint2" type="continuous">        <parent link="link1"/>
         <child link="link2"/>
         <origin xyz="0 0 1.0" rpy="0 0 0"/>
         <axis xyz="0 1 0" />
-    </joint>    <link name="link2">
+    </joint>
+     <link name="link2">
         <xacro:inertial_cylinder mass="0.1" length="1.0" radius="0.05">
             <origin xyz="0 0 0.5" rpy="0 0 0"/>
