Commit message: Pair program with Marguerite: 2_link example that seems to be be working

File: examples/2_link.urdf (robot description, URDF)
Before this commit: robot 2_link, 3 links, 2 joints
Links:
- link link1: geometry 
- link link2: geometry 
Joints:
- joint joint1: axis 0 1 0 -> 0. 1. 0.; origin xyz=0 0 0  rpy=0 0 0 -> xyz=0. 0. 0. rpy=0. 0. 0.; type continuous -> revolute
- joint joint2: axis 0 1 0 -> 0. 1. 0.; origin xyz=0 0 1.0 rpy=0 0 0 -> xyz=0. 0. 1.0 rpy=0. 0. 0.; type continuous -> revolute

Commit message: parallel testing

File: examples/2_link.urdf (robot description, URDF)
Before this commit: robot 2_link, 3 links, 2 joints
Joints:
- joint joint1: axis 0. 1. 0. -> 0. 0. 1.
- joint joint2: axis 0. 1. 0. -> 0. 0. 1.

File: examples/2_link.urdf.xacro (robot description, xacro)
@@ -34,5 +34,6 @@
         </collision>
     </link>
-    <joint name="joint2" type="continuous">        <parent link="link1"/>
+    <joint name="joint2" type="continuous">
+        <parent link="link1"/>
         <child link="link2"/>
         <origin xyz="0 0 1.0" rpy="0 0 0"/>

Commit message: URDF cost (no overloading)- to test

File: examples/2_link.urdf (robot description, URDF)
Before this commit: robot 2_link, 3 links, 2 joints
Joints:
- joint joint1: axis 0. 0. 1. -> 0 1 0; origin xyz=0. 0. 0. rpy=0. 0. 0. -> xyz=0 0 0 rpy=0 0 0
- joint joint2: axis 0. 0. 1. -> 0 1 0; origin xyz=0. 0. 1.0 rpy=0. 0. 0. -> xyz=0 0 1.0 rpy=0 0 0

File: examples/2_link.urdf.xacro (robot description, xacro)
@@ -15,12 +15,12 @@
         <child link="link1"/>
         <origin xyz="0 0 0 " rpy="0 0 0"/>
-        <axis xyz="0 1 0" />
+        <axis xyz="0 0 1" />
     </joint>
     <link name="link1">
         <xacro:inertial_cylinder mass="0.1" length="1.0" radius="0.05">
-            <origin xyz="0 0 0.5" rpy="0 0 0"/>
+            <origin xyz="0.5 0 0" rpy="0 0 0"/>
         </xacro:inertial_cylinder>
         <visual>
-            <origin xyz="0 0 0.5" rpy="0 0 0"/>
+            <origin xyz="0.5 0 0" rpy="0 0 0"/>
             <geometry>
                 <cylinder radius="0.05" length="1.0"/>
@@ -28,5 +28,5 @@
         </visual>
         <collision >
-            <origin xyz="0 0 0.5" rpy="0 0 0"/>
+            <origin xyz="0.5 0 0" rpy="0 0 0"/>
             <geometry>
               <cylinder length="1.0" radius="0.05"/>
@@ -37,13 +37,13 @@
         <parent link="link1"/>
         <child link="link2"/>
-        <origin xyz="0 0 1.0" rpy="0 0 0"/>
-        <axis xyz="0 1 0" />
+        <origin xyz="1 0 0" rpy="0 0 0"/>
+        <axis xyz="0 0 1" />
     </joint>
      <link name="link2">
         <xacro:inertial_cylinder mass="0.1" length="1.0" radius="0.05">
-            <origin xyz="0 0 0.5" rpy="0 0 0"/>
+            <origin xyz="0.5 0 0" rpy="0 0 0"/>
         </xacro:inertial_cylinder>
         <visual>
-            <origin xyz="0 0 0.5" rpy="0 0 0"/>
+            <origin xyz="0.5 0 0" rpy="0 0 0"/>
             <geometry>
                 <cylinder radius="0.05" length="1.0"/>
@@ -51,5 +51,5 @@
         </visual>
         <collision >
-            <origin xyz="0 0 0.5" rpy="0 0 0"/>
+            <origin xyz="0.5 0 0" rpy="0 0 0"/>
             <geometry>
               <cylinder length="1.0" radius="0.05"/>
